Commit message: launch file

File: description/robot_core.xacro (robot description, xacro)
@@ -42,4 +42,7 @@
     </xacro:inertial_box>
 </link>
+<gazebo reference="chassis">
+    <material>Gazebo/White</material>
+</gazebo>
 <!-- LEFT WHEEL -->
 <joint name="left_wheel_joint" type="continuous">
@@ -66,4 +69,7 @@
     </xacro:inertial_cylinder>
 </link>
+<gazebo reference="left_wheel">
+    <material>Gazebo/Blue</material>
+</gazebo>
 <!-- RIGHT WHEEL -->
 <joint name="right_wheel_joint" type="continuous">
@@ -90,4 +96,7 @@
     </xacro:inertial_cylinder>
 </link>
+<gazebo reference="right_wheel">
+    <material>Gazebo/Blue</material>
+</gazebo>
 <!-- CASTER WHEEL -->
 <joint name="caster_wheel_joint" type="fixed">
@@ -113,3 +122,6 @@
     </xacro:inertial_sphere>
 </link>
+<gazebo reference="caster_wheel">
+    <material>Gazebo/Black</material>
+</gazebo>
 </robot>
